File: pcb/ITEA_STM32F030R8T6.sch (KiCad schematic (older format))
At the start: 6 parts

Commit message: Adding backlight pin to schematics
Connections:
- net LCD_BACKLIGHT: now reaches U?.41 (RCC_MCO/TIM1_CH1/USART1_CK/PA8)
Changed lines of the file:
@@
 Wire Notes Line
 	11050 4950 11050 4900
+Text GLabel 7550 2950 2    60   Input ~ 0
+LCD_BACKLIGHT
+Wire Wire Line
+	7150 2950 7550 2950
 $EndSCHEMATC
